File: KiCad_Remote/KiCad_Remote.kicad_pcb (KiCad board)
At the start: 0 parts

Commit message: Update KiCad remote PCB layout
Parts:
- added A1: Arduino_Nano_v3.x, Module:Arduino_Nano_WithMountingHoles, F.Cu at (143.5, 96.0)
- added C1: 10u, Capacitor_THT:CP_Radial_D6.3mm_P2.50mm, F.Cu at (150.5, 52.8)
- added C2: 100n, Capacitor_THT:C_Disc_D3.4mm_W2.1mm_P2.50mm, F.Cu at (158.5, 52.8)
- added C3: 100n, Capacitor_THT:C_Disc_D3.4mm_W2.1mm_P2.50mm, F.Cu at (123.0, 91.5)
- added H1: MountingHole, MountingHole:MountingHole_3.2mm_M3, F.Cu at (171.5, 49.0)
- added H2: MountingHole, MountingHole:MountingHole_3.2mm_M3, F.Cu at (99.5, 106.0)
- added H3: MountingHole, MountingHole:MountingHole_3.2mm_M3, F.Cu at (171.5, 106.0)
- added H4: MountingHole, MountingHole:MountingHole_3.2mm_M3, F.Cu at (99.5, 49.0)
- added J2: Screw_Terminal_01x04, TerminalBlock:TerminalBlock_MaiXu_MX126-5.0-04P_1x04_P5.00mm, F.Cu at (106.5, 91.8)
- added J3: Screw_Terminal_01x07, TerminalBlock:TerminalBlock_MaiXu_MX126-5.0-07P_1x07_P5.00mm, F.Cu at (167.5, 58.5)
- added SW1: SW_Nidec_CAS-120A1, Button_Switch_THT:SW_Slide-03_Wuerth-WS-SLTV_10x2.5x6.4_P2.54mm, F.Cu at (125.5, 103.0)
Routing:
- net /SW: track 0.00 -> 123.1 mm
- net Net-(J3-Pin_7): track 0.00 -> 73.0 mm
- net Net-(A1-D13): track 0.00 -> 65.6 mm
- net Net-(A1-3V3): track 0.00 -> 46.1 mm
- net Net-(A1-D7): track 0.00 -> 34.6 mm
- net Net-(A1-D12): track 0.00 -> 33.7 mm
- net /VRx: track 0.00 -> 27.5 mm
- net Net-(A1-D11): track 0.00 -> 24.2 mm
- net Net-(A1-D5): track 0.00 -> 24.1 mm
- net /GND: track 0.00 -> 22.7 mm
- net /+5V: track 0.00 -> 22.5 mm
- net Net-(A1-VIN): track 0.00 -> 15.4 mm
Other:
- board outline added: 80 x 65 mm
- copper layers 0 -> 2
