File: KiCad_Remote/KiCad_Remote.kicad_sch (KiCad schematic)
At the start: 2 parts, among them J1 Conn_01x05

Commit message: Update KiCad remote PCB layout
Parts:
- removed A1: Arduino_Nano_v2.x, Module:Arduino_Nano, symbol MCU_Module:Arduino_Nano_v2.x
- added A1: Arduino_Nano_v3.x, Module:Arduino_Nano_WithMountingHoles, symbol MCU_Module:Arduino_Nano_v3.x
- added BT1: Battery_Cell, symbol Device:Battery_Cell
- added C1: 10u, Capacitor_THT:CP_Radial_D6.3mm_P2.50mm, symbol Device:C_Polarized
- added C2, C3: 100n, Capacitor_THT:C_Disc_D3.4mm_W2.1mm_P2.50mm, symbol Device:C
- added H1, H2, H3, H4: MountingHole, MountingHole:MountingHole_3.2mm_M3, symbol Mechanical:MountingHole
- added J2: Screw_Terminal_01x04, TerminalBlock:TerminalBlock_MaiXu_MX126-5.0-04P_1x04_P5.00mm, symbol Connector:Screw_Terminal_01x04
- added J3: Screw_Terminal_01x07, TerminalBlock:TerminalBlock_MaiXu_MX126-5.0-07P_1x07_P5.00mm, symbol Connector:Screw_Terminal_01x07
- added SW1: SW_Nidec_CAS-120A1, Button_Switch_THT:SW_Slide-03_Wuerth-WS-SLTV_10x2.5x6.4_P2.54mm, symbol Switch:SW_Nidec_CAS-120A1
- added U1: NRF24L01_Breakout, RF_Module:nRF24L01_Breakout, symbol RF:NRF24L01_Breakout
Connections:
- net GND: now reaches J1.1 (Pin_1)
- net GND: now also A1.29 (GND), C3.1, J2.1 (Pin_1)
- net +5V: now reaches J1.2 (Pin_2)
- net +5V: now also A1.27 (+5V), J2.2 (Pin_2)
- net VRx: now reaches J1.3 (Pin_3)
- net VRx: now also A1.19 (A0), J2.3 (Pin_3)
- net SW: now reaches J1.5 (Pin_5)
- net SW: now also A1.5 (D2), J2.4 (Pin_4)
- new net: A1.17 (3V3), C1.1, C2.1, J3.1 (Pin_1), U1.2 (VCC)
- new net: A1.4 (GND), C1.2, C2.2, J3.7 (Pin_7), U1.1 (GND)
- new net: A1.30 (VIN), BT1.1 (+), C3.2, SW1.2 (B)
- new net: BT1.2 (-), SW1.3 (A)
- new net: A1.14 (D11), J3.2 (Pin_2), U1.6 (MOSI)
- new net: A1.15 (D12), J3.3 (Pin_3), U1.7 (MISO)
- new net: A1.16 (D13), J3.4 (Pin_4), U1.5 (SCK)
- new net: A1.8 (D5), J3.5 (Pin_5), U1.4 (~{CSN})
- new net: A1.10 (D7), J3.6 (Pin_6), U1.3 (CE)
- no-connect marks 0 -> 21
