File: KiCad_Remote/Remote.kicad_sch (KiCad schematic)
At the start: 9 parts, among them J1 Screw_Terminal_01x04, SW1 SW_Wuerth_450301014042, U1 NRF24L01_Breakout

Commit message: Finished Remote
Remote is finished and need review
Parts:
- added H1, H2, H3, H4: MountingHole, MountingHole:MountingHole_3.2mm_M3, symbol Mechanical:MountingHole
- added J2: Screw_Terminal_01x02, TerminalBlock:TerminalBlock_MaiXu_MX126-5.0-02P_1x02_P5.00mm, symbol Connector:Screw_Terminal_01x02
- added NT1, NT2: NetTie_2, LibraryNewHoleSize:NetTie_1.6mm, symbol Device:NetTie_2
- U1: footprint TerminalBlock:TerminalBlock_MaiXu_MX126-5.0-08P_1x08_P5.00mm -> LibraryNewHoleSize:nRF24L01_Breakout
- renumbered C8 to C2, C9 to C3
Connections:
- net 5: now also J1.3 (Pin_3); no longer J1.2 (Pin_2)
- net Botton_Joystick: now also J1.4 (Pin_4); no longer J1.3 (Pin_3)
- net GND: now also J2.1 (Pin_1), NT1.2, NT2.2; no longer A1.29 (GND), C1.1, C2.2, C3.2, U1.1 (GND)
- net Joystick_X: now also A1.20 (A1), J1.2 (Pin_2); no longer A1.19 (A0), J1.4 (Pin_4)
- net Speed: now also A1.19 (A0); no longer A1.20 (A1)
- net VCC: now also J2.2 (Pin_2)
- new net GND_Arduino: A1.29 (GND), C1.1, NT1.1
- new net GND_NRF: C2.2, C3.2, NT2.1, U1.1 (GND)
Other:
- moved on the sheet: C2, C3, R1, R2, SW1, U1
